File: 2wd/2wd.brd (EAGLE design)
At the start: 100 x 80 mm, 10 parts

Commit message: Start adding power control
Parts:
- added IC1: REG1118, burr-brown:SOT223
- added J1: (no value), con-jack:SPC4077
Connections:
- removed net 3V3: U$5.JP1.8
- removed net 5V: U$5.JP2.8
- new net N$10: IC1.1, U$5.JP2.8
- new net N$11: J1.2, U$5.JP1.8
- new net N$9: IC1.3, U$4.OUT+
- net GND: now also IC1.2, J1.1, U$4.OUT-
- net VCC: now also J1.3
Routing:
- net N$9: track 0.00 -> 70.8 mm
- net N$11: track 0.00 -> 68.7 mm
- net GND: track 124.8 -> 189.4 mm
- net VCC: track 131.1 -> 187.7 mm
- net N$10: track 0.00 -> 18.9 mm
- net N$6: track 92.1 -> 81.0 mm
- net N$3: track 79.7 -> 81.2 mm
