File: 2wd/2wd.sch (EAGLE design)
At the start: 10 parts

Commit message: Start adding power control
Parts:
- added IC1: REG1118, burr-brown:REG1118
- added J1: (no value), con-jack:JACK-PLUG0
Connections:
- new net N$10: IC1.VOUT, U$5.5V
- new net N$11: J1.2, U$5.3V3
- new net N$9: IC1.VIN, U$4.OUT+
- net GND: now also IC1.GND, J1.1, U$4.OUT-
- net VCC: now also J1.3
Changed lines of the file:
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@@
 <part name="U$8" library="diy-modules" deviceset="BATTERY-LI-MH12210" device=""/>
 <part name="U$9" library="diy-modules" deviceset="BATTERY-LI-MH12210" device=""/>
+<part name="IC1" library="burr-brown" deviceset="REG1118" device=""/>
+<part name="J1" library="con-jack" deviceset="JACK-PLUG" device="0"/>
 </parts>
 <sheets>
@@
 <instance part="U$8" gate="G$1" x="175.26" y="132.08" rot="R180"/>
 <instance part="U$9" gate="G$1" x="210.82" y="109.22" rot="R180"/>
+<instance part="IC1" gate="G$1" x="48.26" y="149.86"/>
+<instance part="J1" gate="G$1" x="15.24" y="25.4"/>
 </instances>
 <busses>
@@
 <pinref part="U$1" gate="G$1" pin="IN+"/>
 <wire x1="203.2" y1="40.64" x2="203.2" y2="48.26" width="0.1524" layer="91"/>
+<pinref part="J1" gate="G$1" pin="3"/>
+<wire x1="20.32" y1="27.94" x2="88.9" y2="27.94" width="0.1524" layer="91"/>
+<wire x1="88.9" y1="27.94" x2="88.9" y2="40.64" width="0.1524" layer="91"/>
+<junction x="88.9" y="40.64"/>
 </segment>
 </net>
@@
 <pinref part="U$5" gate="G$1" pin="GND"/>
 <wire x1="76.2" y1="63.5" x2="66.04" y2="63.5" width="0.1524" layer="91"/>
+</segment>
+<segment>
+<pinref part="IC1" gate="G$1" pin="GND"/>
+<wire x1="48.26" y1="137.16" x2="48.26" y2="132.08" width="0.1524" layer="91"/>
+<label x="48.26" y="132.08" size="1.778" layer="95"/>
+</segment>
+<segment>
+<pinref part="U$4" gate="G$1" pin="OUT-"/>
+<wire x1="104.14" y1="81.28" x2="104.14" y2="88.9" width="0.1524" layer="91"/>
+<label x="104.14" y="86.36" size="1.778" layer="95"/>
+</segment>
+<segment>
+<pinref part="J1" gate="G$1" pin="1"/>
+<wire x1="20.32" y1="22.86" x2="30.48" y2="22.86" width="0.1524" layer="91"/>
+<wire x1="30.48" y1="22.86" x2="30.48" y2="17.78" width="0.1524" layer="91"/>
+<label x="30.48" y="17.78" size="1.778" layer="95"/>
 </segment>
 </net>
@@
 </segment>
 </net>
+<net name="N$9" class="0">
+<segment>
+<pinref part="U$4" gate="G$1" pin="OUT+"/>
+<wire x1="88.9" y1="81.28" x2="88.9" y2="111.76" width="0.1524" layer="91"/>
+<pinref part="IC1" gate="G$1" pin="VIN"/>
+<wire x1="88.9" y1="111.76" x2="35.56" y2="111.76" width="0.1524" layer="91"/>
+<wire x1="35.56" y1="111.76" x2="35.56" y2="149.86" width="0.1524" layer="91"/>
+</segment>
+</net>
+<net name="N$10" class="0">
+<segment>
+<pinref part="IC1" gate="G$1" pin="VOUT"/>
+<wire x1="60.96" y1="149.86" x2="71.12" y2="149.86" width="0.1524" layer="91"/>
+<wire x1="71.12" y1="149.86" x2="71.12" y2="60.96" width="0.1524" layer="91"/>
+<pinref part="U$5" gate="G$1" pin="5V"/>
+<wire x1="71.12" y1="60.96" x2="66.04" y2="60.96" width="0.1524" layer="91"/>
+</segment>
+</net>
+<net name="N$11" class="0">
+<segment>
+<pinref part="J1" gate="G$1" pin="2"/>
+<wire x1="20.32" y1="25.4" x2="30.48" y2="25.4" width="0.1524" layer="91"/>
+<pinref part="U$5" gate="G$1" pin="3V3"/>
+<wire x1="30.48" y1="25.4" x2="30.48" y2="60.96" width="0.1524" layer="91"/>
+</segment>
+</net>
